File: Hardware/PCB.brd (EAGLE design)
At the start: 170.2 x 111.2 mm, 103 parts, among them IC1 BD5229G-TR, IC4 XC6220A331MR-G, J1 FH34SRJ-24S-0.5SH_99_, J3 QWIIC_RIGHT_ANGLE, J4 112A-TAAR-R03_ATTEND, Q1 20V/4.2A/52mΩ/1.4W, Q2 20V/4.2A/52mΩ/1.4W, Q3 SI1308EDL-T1-GE3, U1 W25Q512JVEIQ, U2 ESP32-C6-WROOM-1-N8, U3 DS3231SN#, U4 MAX17048G+T10

Commit message: Solved all issues
Parts:
- EPD_C5: value 1uF/50V -> 0.1uF/50V
- moved R2-USB1 1.63 mm to (157.0, 54.2)
- moved TP11 0.50 mm to (48.5, 3.50)
- moved TP12 0.50 mm to (53.6, 3.50)
- moved TP17 0.50 mm to (58.7, 3.60)
- moved TP7 0.50 mm to (36.0, 3.48)
- moved TP8 0.50 mm to (40.2, 3.48)
- moved TP9 0.50 mm to (44.4, 3.58)
Routing:
- net 3V3: track 406.6 -> 407.8 mm
- net N$1: track 7.30 -> 8.31 mm
- net EPD_RST: track 110.3 -> 109.6 mm
- net GND: track 673.3 -> 673.9 mm
- net MOSI: track 210.3 -> 209.8 mm
Other:
- board text added: "3V3"
- board text added: "EPD_3V3"
- board text added: "EPD_3V3_C"
- board text added: "EPD_BUSY"
- board text added: "EPD_CS"
- board text added: "EPD_DC"
- board text added: "EPD_RST"
- board text added: "GND"
- board text added: "INT_RTC"
- board text added: "L1"
- board text added: "MISO"
- board text added: "MOSI"
- board text added: "RX"
- board text added: "SCK"
- board text added: "TX"
- board text added: "VBAT"
- board text added: "VBUS"
