File: Hardware/Schematic.sch (EAGLE design)
At the start: 103 parts, among them IC1 BD5229G-TR, IC4 XC6220A331MR-G, J1 FH34SRJ-24S-0.5SH_99_, J2 SAMACSYS_PARTS_USB4110-GF-A, J3 QWIIC_RIGHT_ANGLE, J4 112A-TAAR-R03_ATTEND, Q1 20V/4.2A/52mΩ/1.4W, Q2 20V/4.2A/52mΩ/1.4W, Q3 SI1308EDL-T1-GE3, U1 W25Q512JVEIQ, U2 ESP32-C6-WROOM-1-N8, U3 DS3231SN#, U4 MAX17048G+T10

Commit message: Solved all issues
Parts:
- EPD_C5: value 1uF/50V -> 0.1uF/50V
Other:
- note added: "DMG2305UX-7"
- note added: "drawn by: Robert Damian"
Changed lines of the file:
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@@
 <setting verticaltext="up"/>
 </settings>
-<grid distance="0.1" unitdist="inch" unit="inch" style="lines" multiple="1" display="no" altdistance="0.01" altunitdist="inch" altunit="inch"/>
+<grid distance="0.05" unitdist="inch" unit="inch" style="lines" multiple="1" display="yes" altdistance="0.01" altunitdist="inch" altunit="inch"/>
 <layers>
 <layer number="1" name="Top" color="4" fill="1" visible="no" active="no"/>
@@
 <part name="EPD_C7" library="DeskAssistant v19 v1" library_urn="urn:adsk.wipprod:fs.file:vf.QwFj3SzAQTmJBbbHAlSUAQ" deviceset="EAGLE-LTSPICE_C" device="C0402" value="1uF/50V"/>
 <part name="EPD_C6" library="DeskAssistant v19 v1" library_urn="urn:adsk.wipprod:fs.file:vf.QwFj3SzAQTmJBbbHAlSUAQ" deviceset="EAGLE-LTSPICE_C" device="C0402" value="1uF/50V"/>
-<part name="EPD_C5" library="DeskAssistant v19 v1" library_urn="urn:adsk.wipprod:fs.file:vf.QwFj3SzAQTmJBbbHAlSUAQ" deviceset="EAGLE-LTSPICE_C" device="C0402" value="1uF/50V"/>
+<part name="EPD_C5" library="DeskAssistant v19 v1" library_urn="urn:adsk.wipprod:fs.file:vf.QwFj3SzAQTmJBbbHAlSUAQ" deviceset="EAGLE-LTSPICE_C" device="C0402" value="0.1uF/50V"/>
 <part name="SUPPLY27" library="DeskAssistant v19 v1" library_urn="urn:adsk.wipprod:fs.file:vf.QwFj3SzAQTmJBbbHAlSUAQ" deviceset="GND-BAR" device="" value="GND"/>
 <part name="SUPPLY28" library="DeskAssistant v19 v1" library_urn="urn:adsk.wipprod:fs.file:vf.QwFj3SzAQTmJBbbHAlSUAQ" deviceset="GND-BAR" device="" value="GND"/>
@@
 <text x="171.45" y="-162.56" size="3.81" layer="97">SPI ESD Protection Lines</text>
 <text x="254" y="-162.56" size="3.81" layer="97">External NORFlash64MB</text>
+<text x="162.56" y="7.62" size="1.778" layer="95">DMG2305UX-7</text>
+<text x="85.09" y="-106.68" size="1.778" layer="95" rot="R90">DMG2305UX-7</text>
+<text x="308.61" y="-203.2" size="2.413" layer="94">drawn by: Robert Damian</text>
 </plain>
 <instances>
@@
 </instance>
 <instance part="Q1" gate="G$1" x="157.48" y="10.16" smashed="yes">
-<attribute name="NAME" x="162.56" y="10.16" size="1.778" layer="95" font="vector"/>
-<attribute name="VALUE" x="162.56" y="7.62" size="1.778" layer="96" font="vector"/>
+<attribute name="NAME" x="162.56" y="12.7" size="1.778" layer="95" font="vector"/>
+<attribute name="VALUE" x="162.56" y="10.16" size="1.778" layer="96" font="vector"/>
 </instance>
 <instance part="R1_PWRUSB" gate="G$1" x="139.7" y="-2.54" smashed="yes" rot="R90">
@@
 <instance part="Q2" gate="G$1" x="77.47" y="-104.14" smashed="yes">
 <attribute name="NAME" x="82.55" y="-106.68" size="1.778" layer="95" font="vector" rot="R90"/>
-<attribute name="VALUE" x="85.09" y="-106.68" size="1.778" layer="96" font="vector" rot="R90"/>
+<attribute name="VALUE" x="87.63" y="-106.68" size="1.778" layer="96" font="vector" rot="R90"/>
 </instance>
 <instance part="SENSOR2" gate="G$1" x="119.38" y="-105.41" smashed="yes">
@@
 </instance>
 <instance part="C6" gate="G$1" x="254" y="-114.3" smashed="yes">
-<attribute name="NAME" x="139.319" y="502.666" size="1.778" layer="95" rot="R270"/>
-<attribute name="VALUE" x="256.794" y="-112.649" size="1.778" layer="96" rot="R270"/>
+<attribute name="NAME" x="251.079" y="-116.586" size="1.778" layer="95" rot="R90"/>
+<attribute name="VALUE" x="258.699" y="-119.126" size="1.778" layer="96" rot="R90"/>
 </instance>
 <instance part="SUPPLY43" gate="G$1" x="247.65" y="-125.73" smashed="yes">
@@
 <wire x1="139.7" y1="7.62" x2="139.7" y2="13.97" width="0.1524" layer="91"/>
 <wire x1="139.7" y1="2.54" x2="139.7" y2="7.62" width="0.1524" layer="91"/>
-<label x="139.7" y="10.16" size="1.27" layer="95" rot="R90" xref="yes"/>
+<label x="139.7" y="13.97" size="1.27" layer="95" rot="R90" xref="yes"/>
 <junction x="142.24" y="7.62"/>
 <junction x="139.7" y="7.62"/>
